File: Nano-keyboard/Nano-keyboard.kicad_sch (KiCad schematic)
At the start: 39 parts, among them U2 ESP32-WROOM-32

Commit message: Minor schematic changes
Parts:
- removed LED12: LRTBGVSR-U4V2-JW+A6BB-D8+S2U2-7Z-20-S, lib:LRTBGVSRU4V2JWA6BBD8S2U27Z20S, symbol custom-keyboard:LRTBGVSR-U4V2-JW+A6BB-D8+S2U2-7Z-20-S

Commit message: 3D Switch Models
Parts:
- removed B1, B10, B11, B12, B2, B3, B4, B5, B6, B7, B8, B9: Cherry_Switch_1U_PCB, Button_Switch_Keyboard:SW_Cherry_MX_1.00u_PCB, symbol CustomButton:Cherry_Switch_1U_PCB
- added B1, B10, B11, B12, B2, B3, B4, B5, B6, B7, B8, B9: Cherry_Switch_1U_PCB, lib:SW_Cherry_MX_1.00u_PCB, symbol custom-keyboard:Cherry_Switch_1U_PCB
Connections:
- net COL1: now also B1.2, B5.2, B9.2
- net COL2: now also B10.2, B2.2, B6.2
- net COL3: now also B11.2, B3.2, B7.2
- net COL4: now also B12.2, B4.2, B8.2
- net at D1.2 (A): now also B1.1
- net at D6.2 (A): now also B6.1
- net at D7.2 (A): now also B7.1
- net at D11.2 (A): now also B11.1
- net at D10.2 (A): now also B10.1
- net at D12.2 (A): now also B12.1
- net at D5.2 (A): now also B5.1
- net at D4.2 (A): now also B4.1
- net at D3.2 (A): now also B3.1
- net at D8.2 (A): now also B8.1
- net at D9.2 (A): now also B9.1
- net at D2.2 (A): now also B2.1

Commit message: Minor changes
Parts:
- removed B0: Cherry_Switch_1U_PCB, Button_Switch_Keyboard:SW_Cherry_MX_1.00u_PCB, symbol CustomButton:Cherry_Switch_1U_PCB
- added B0: Cherry_Switch_1U_PCB, lib:SW_Cherry_MX_1.00u_PCB, symbol custom-keyboard:Cherry_Switch_1U_PCB
- added U1, U3, U4: QBC847BL, lib:SOT96P237X111-3N, symbol custom-keyboard:QBC847BL
Connections:
- net +3V3: now also B0.1, U1.3 (E), U3.3 (E), U4.3 (E)
- net ANODE_B: now also U4.2 (C)
- net ANODE_G: now also U3.2 (C)
- net ANODE_R: now also U1.2 (C)
- net FUNC: now also B0.2
Changed lines of the file:
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@@
   (junction (at 179.07 38.1) (diameter 0) (color 0 0 0 0)
   )
+  (junction (at 170.688 127.254) (diameter 0) (color 0 0 0 0)
+  )
   (junction (at 26.924 100.076) (diameter 0) (color 0 0 0 0)
   )
@@
   (junction (at 189.23 59.69) (diameter 0) (color 0 0 0 0)
   )
+  (junction (at 170.688 113.03) (diameter 0) (color 0 0 0 0)
+  )
   (junction (at 175.26 55.88) (diameter 0) (color 0 0 0 0)
   )
@@
     (stroke (width 0) (type default) (color 0 0 0 0))
   )
+  (wire (pts (xy 167.132 113.03) (xy 167.132 113.284))
+    (stroke (width 0) (type default) (color 0 0 0 0))
+  )
   (wire (pts (xy 27.178 181.102) (xy 28.956 181.102))
     (stroke (width 0) (type default) (color 0 0 0 0))
@@
     (stroke (width 0) (type default) (color 0 0 0 0))
   )
+  (wire (pts (xy 170.688 113.03) (xy 167.132 113.03))
+    (stroke (width 0) (type default) (color 0 0 0 0))
+  )
+  (wire (pts (xy 167.132 137.414) (xy 177.038 137.414))
+    (stroke (width 0) (type default) (color 0 0 0 0))
+  )
   (wire (pts (xy 26.924 155.956) (xy 26.924 161.036))
     (stroke (width 0) (type default) (color 0 0 0 0))
@@
     (stroke (width 0) (type default) (color 0 0 0 0))
   )
+  (wire (pts (xy 167.132 123.444) (xy 177.038 123.444))
+    (stroke (width 0) (type default) (color 0 0 0 0))
+  )
   (wire (pts (xy 53.594 80.01) (xy 44.196 80.01))
     (stroke (width 0) (type default) (color 0 0 0 0))
@@
     (stroke (width 0) (type default) (color 0 0 0 0))
   )
+  (wire (pts (xy 170.688 127.254) (xy 170.688 113.03))
+    (stroke (width 0) (type default) (color 0 0 0 0))
+  )
   (wire (pts (xy 53.848 150.876) (xy 44.45 150.876))
     (stroke (width 0) (type default) (color 0 0 0 0))
@@
     (stroke (width 0) (type default) (color 0 0 0 0))
   )
+  (wire (pts (xy 167.132 150.114) (xy 177.038 150.114))
+    (stroke (width 0) (type default) (color 0 0 0 0))
+  )
   (wire (pts (xy 54.102 176.022) (xy 44.704 176.022))
     (stroke (width 0) (type default) (color 0 0 0 0))
   )
+  (wire (pts (xy 170.688 139.954) (xy 170.688 127.254))
+    (stroke (width 0) (type default) (color 0 0 0 0))
+  )
   (wire (pts (xy 26.924 140.716) (xy 28.702 140.716))
     (stroke (width 0) (type default) (color 0 0 0 0))
@@
     (stroke (width 0) (type default) (color 0 0 0 0))
   )
+  (wire (pts (xy 167.132 127.254) (xy 170.688 127.254))
+    (stroke (width 0) (type default) (color 0 0 0 0))
+  )
   (wire (pts (xy 175.26 55.88) (xy 185.42 55.88))
     (stroke (width 0) (type default) (color 0 0 0 0))
@@
   )
   (wire (pts (xy 85.344 29.21) (xy 75.946 29.21))
+    (stroke (width 0) (type default) (color 0 0 0 0))
+  )
+  (wire (pts (xy 167.132 139.954) (xy 170.688 139.954))
     (stroke (width 0) (type default) (color 0 0 0 0))
   )
@@
     (effects (font (size 1.27 1.27)) (justify right bottom))
   )
+  (label "ANODE_G" (at 177.038 137.414 180)
+    (effects (font (size 1.27 1.27)) (justify right bottom))
+  )
   (label "ANODE_G" (at 85.852 94.742 180)
     (effects (font (size 1.27 1.27)) (justify right bottom))
@@
   )
   (label "ANODE_B" (at 53.848 161.036 180)
+    (effects (font (size 1.27 1.27)) (justify right bottom))
+  )
+  (label "ANODE_R" (at 177.038 123.444 180)
     (effects (font (size 1.27 1.27)) (justify right bottom))
   )
@@
   )
   (label "ANODE_B" (at 85.344 39.37 180)
+    (effects (font (size 1.27 1.27)) (justify right bottom))
+  )
+  (label "ANODE_B" (at 177.038 150.114 180)
     (effects (font (size 1.27 1.27)) (justify right bottom))
   )
@@
     )
     (property "Datasheet" "" (id 3) (at 26.67 80.01 0)
+      (effects (font (size 1.27 1.27)) hide)
+    )
+    (pin "1")
+  )
+  (symbol (lib_id "power:+3.3V") (at 170.688 113.03 0) (unit 1)
+    (in_bom yes) (on_board yes) (fields_autoplaced)
+    (property "Reference" "#PWR013" (id 0) (at 170.688 116.84 0)
+      (effects (font (size 1.27 1.27)) hide)
+    )
+    (property "Value" "+3.3V" (id 1) (at 170.688 107.95 0))
+    (property "Footprint" "" (id 2) (at 170.688 113.03 0)
+      (effects (font (size 1.27 1.27)) hide)
+    )
+    (property "Datasheet" "" (id 3) (at 170.688 113.03 0)
       (effects (font (size 1.27 1.27)) hide)
     )
@@
     (pin "C2")
     (pin "C3")
+  )
+  (symbol (lib_id "custom-keyboard:QBC847BL") (at 165.1 118.11 0) (unit 1)
+    (in_bom yes) (on_board yes) (fields_autoplaced)
+    (property "Reference" "U1" (id 0) (at 170.18 117.0939 0)
+      (effects (font (size 1.27 1.27)) (justify left))
+    )
+    (property "Value" "QBC847BL" (id 1) (at 170.18 119.6339 0)
+      (effects (font (size 1.27 1.27)) (justify left))
+    )
+    (property "Footprint" "lib:SOT96P237X111-3N" (id 2) (at 178.816 123.444 0)
+      (effects (font (size 1.27 1.27)) hide)
+    )
+    (property "Datasheet" "" (id 3) (at 165.1 118.11 0)
+      (effects (font (size 1.27 1.27)) hide)
+    )
+    (pin "1")
+    (pin "2")
+    (pin "3")
   )
   (symbol (lib_id "custom-keyboard:Cherry_Switch_1U_PCB") (at 194.31 43.18 90) (unit 1)
@@
     (pin "C3")
   )
-  (symbol (lib_id "CustomButton:Cherry_Switch_1U_PCB") (at 125.73 29.21 0) (unit 1)
-    (in_bom yes) (on_board yes) (fields_autoplaced)
-    (property "Reference" "B0" (id 0) (at 125.73 24.13 0))
-    (property "Value" "Cherry_Switch_1U_PCB" (id 1) (at 124.4601 30.48 90)
-      (effects (font (size 1.27 1.27)) (justify right) hide)
-    )
-    (property "Footprint" "Button_Switch_Keyboard:SW_Cherry_MX_1.00u_PCB" (id 2) (at 130.81 30.48 0)
-      (effects (font (size 1.27 1.27)) hide)
-    )
-    (property "Datasheet" "" (id 3) (at 125.73 29.21 0)
-      (effects (font (size 1.27 1.27)) hide)
-    )
-    (pin "1")
-    (pin "2")
-  )
   (symbol (lib_id "power:GND") (at 26.924 161.036 0) (unit 1)
     (in_bom yes) (on_board yes) (fields_autoplaced)
@@
     (pin "2")
   )
+  (symbol (lib_id "custom-keyboard:QBC847BL") (at 165.1 144.78 0) (unit 1)
+    (in_bom yes) (on_board yes) (fields_autoplaced)
+    (property "Reference" "U4" (id 0) (at 170.18 143.7639 0)
+      (effects (font (size 1.27 1.27)) (justify left))
+    )
+    (property "Value" "QBC847BL" (id 1) (at 170.18 146.3039 0)
+      (effects (font (size 1.27 1.27)) (justify left))
+    )
+    (property "Footprint" "lib:SOT96P237X111-3N" (id 2) (at 178.816 150.114 0)
+      (effects (font (size 1.27 1.27)) hide)
+    )
+    (property "Datasheet" "" (id 3) (at 165.1 144.78 0)
+      (effects (font (size 1.27 1.27)) hide)
+    )
+    (pin "1")
+    (pin "2")
+    (pin "3")
+  )
   (symbol (lib_name "LRTBGVSR-U4V2-JW+A6BB-D8+S2U2-7Z-20-S_1") (lib_id "custom-keyboard:LRTBGVSR-U4V2-JW+A6BB-D8+S2U2-7Z-20-S") (at 33.274 74.676 0) (unit 1)
     (in_bom yes) (on_board yes)
@@
     (pin "C3")
   )
+  (symbol (lib_id "custom-keyboard:QBC847BL") (at 165.1 132.08 0) (unit 1)
+    (in_bom yes) (on_board yes) (fields_autoplaced)
+    (property "Reference" "U3" (id 0) (at 170.18 131.0639 0)
+      (effects (font (size 1.27 1.27)) (justify left))
+    )
+    (property "Value" "QBC847BL" (id 1) (at 170.18 133.6039 0)
+      (effects (font (size 1.27 1.27)) (justify left))
+    )
+    (property "Footprint" "lib:SOT96P237X111-3N" (id 2) (at 178.816 137.414 0)
+      (effects (font (size 1.27 1.27)) hide)
+    )
+    (property "Datasheet" "" (id 3) (at 165.1 132.08 0)
+      (effects (font (size 1.27 1.27)) hide)
+    )
+    (pin "1")
+    (pin "2")
+    (pin "3")
+  )
   (symbol (lib_id "power:GND") (at 26.924 100.076 0) (unit 1)
     (in_bom yes) (on_board yes) (fields_autoplaced)
@@
     )
     (property "Datasheet" "http://www.vishay.com/docs/85622/1n914.pdf" (id 3) (at 185.42 52.07 0)
+      (effects (font (size 1.27 1.27)) hide)
+    )
+    (pin "1")
+    (pin "2")
+  )
+  (symbol (lib_id "custom-keyboard:Cherry_Switch_1U_PCB") (at 125.73 29.21 0) (unit 1)
+    (in_bom yes) (on_board yes) (fields_autoplaced)
+    (property "Reference" "B0" (id 0) (at 125.73 24.13 0))
+    (property "Value" "Cherry_Switch_1U_PCB" (id 1) (at 125.73 24.13 0)
+      (effects (font (size 1.27 1.27)) hide)
+    )
+    (property "Footprint" "lib:SW_Cherry_MX_1.00u_PCB" (id 2) (at 130.81 30.48 0)
+      (effects (font (size 1.27 1.27)) hide)
+    )
+    (property "Datasheet" "" (id 3) (at 125.73 29.21 0)
       (effects (font (size 1.27 1.27)) hide)
     )
@@
       (reference "#PWR012") (unit 1) (value "GND") (footprint "")
     )
+    (path "/07fc269a-0aca-4937-9fc5-5cd6b5a06b6c"
+      (reference "#PWR013") (unit 1) (value "+3.3V") (footprint "")
+    )
     (path "/e95b1d8e-2e4e-4877-9121-2ee2965866b4"
       (reference "#PWR0101") (unit 1) (value "+3.3V") (footprint "")
     )
-    (path "/7fc01d77-2b58-46d3-be57-a8f53dbe3176"
-      (reference "B0") (unit 1) (value "Cherry_Switch_1U_PCB") (footprint "Button_Switch_Keyboard:SW_Cherry_MX_1.00u_PCB")
+    (path "/e891b433-8f8c-451a-9a1f-eebc6bd34030"
+      (reference "B0") (unit 1) (value "Cherry_Switch_1U_PCB") (footprint "lib:SW_Cherry_MX_1.00u_PCB")
     )
     (path "/6176909e-4118-4be8-ab95-c4bd46ff7347"
@@
       (reference "LED11") (unit 1) (value "LRTBGVSR-U4V2-JW+A6BB-D8+S2U2-7Z-20-S") (footprint "lib:LRTBGVSRU4V2JWA6BBD8S2U27Z20S")
     )
+    (path "/1ff22ddb-0012-441d-8a0b-04f938747f91"
+      (reference "U1") (unit 1) (value "QBC847BL") (footprint "lib:SOT96P237X111-3N")
+    )
     (path "/5daf0f2c-a4b4-4b3d-9961-01231612289d"
       (reference "U2") (unit 1) (value "ESP32-WROOM-32") (footprint "RF_Module:ESP32-WROOM-32")
     )
-  )
+    (path "/c875fac1-49a7-4dcd-9a7a-05bc0a9ca91a"
+      (reference "U3") (unit 1) (value "QBC847BL") (footprint "lib:SOT96P237X111-3N")
+    )
+    (path "/aa91d7bc-c62e-4dc0-bf06-c00a6378f5d9"
+      (reference "U4") (unit 1) (value "QBC847BL") (footprint "lib:SOT96P237X111-3N")
+    )
+  )

Commit message: Diode Changes
Parts:
- D1, D10, D11, D12, D3, D4, D5, D6, D7, D8, D9: footprint Diode_THT:D_DO-35_SOD27_P7.62mm_Horizontal -> Diode_THT:D_DO-35_SOD27_P3.81mm_Vertical_AnodeUp
Changed lines of the file:
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@@
       (effects (font (size 1.27 1.27)) (justify right) hide)
     )
-    (property "Footprint" "Diode_THT:D_DO-35_SOD27_P7.62mm_Horizontal" (id 2) (at 189.865 73.66 0)
+    (property "Footprint" "Diode_THT:D_DO-35_SOD27_P3.81mm_Vertical_AnodeUp" (id 2) (at 189.865 73.66 0)
       (effects (font (size 1.27 1.27)) hide)
     )
@@
       (effects (font (size 1.27 1.27)) (justify right) hide)
     )
-    (property "Footprint" "Diode_THT:D_DO-35_SOD27_P7.62mm_Horizontal" (id 2) (at 189.865 95.25 0)
+    (property "Footprint" "Diode_THT:D_DO-35_SOD27_P3.81mm_Vertical_AnodeUp" (id 2) (at 189.865 95.25 0)
       (effects (font (size 1.27 1.27)) hide)
     )
@@
       (effects (font (size 1.27 1.27)) (justify right) hide)
     )
-    (property "Footprint" "Diode_THT:D_DO-35_SOD27_P7.62mm_Horizontal" (id 2) (at 206.375 95.25 0)
+    (property "Footprint" "Diode_THT:D_DO-35_SOD27_P3.81mm_Vertical_AnodeUp" (id 2) (at 206.375 95.25 0)
       (effects (font (size 1.27 1.27)) hide)
     )
@@
       (effects (font (size 1.27 1.27)) (justify right) hide)
     )
-    (property "Footprint" "Diode_THT:D_DO-35_SOD27_P7.62mm_Horizontal" (id 2) (at 179.705 52.07 0)
+    (property "Footprint" "Diode_THT:D_DO-35_SOD27_P3.81mm_Vertical_AnodeUp" (id 2) (at 179.705 52.07 0)
       (effects (font (size 1.27 1.27)) hide)
     )
@@
       (effects (font (size 1.27 1.27)) (justify right) hide)
     )
-    (property "Footprint" "Diode_THT:D_DO-35_SOD27_P7.62mm_Horizontal" (id 2) (at 179.705 73.66 0)
+    (property "Footprint" "Diode_THT:D_DO-35_SOD27_P3.81mm_Vertical_AnodeUp" (id 2) (at 179.705 73.66 0)
       (effects (font (size 1.27 1.27)) hide)
     )
@@
       (effects (font (size 1.27 1.27)) (justify right) hide)
     )
-    (property "Footprint" "Diode_THT:D_DO-35_SOD27_P7.62mm_Horizontal" (id 2) (at 198.755 73.66 0)
+    (property "Footprint" "Diode_THT:D_DO-35_SOD27_P3.81mm_Vertical_AnodeUp" (id 2) (at 198.755 73.66 0)
       (effects (font (size 1.27 1.27)) hide)
     )
@@
       (effects (font (size 1.27 1.27)) (justify right) hide)
     )
-    (property "Footprint" "Diode_THT:D_DO-35_SOD27_P7.62mm_Horizontal" (id 2) (at 198.755 52.07 0)
+    (property "Footprint" "Diode_THT:D_DO-35_SOD27_P3.81mm_Vertical_AnodeUp" (id 2) (at 198.755 52.07 0)
       (effects (font (size 1.27 1.27)) hide)
     )
@@
       (effects (font (size 1.27 1.27)) (justify right) hide)
     )
-    (property "Footprint" "Diode_THT:D_DO-35_SOD27_P7.62mm_Horizontal" (id 2) (at 198.755 95.25 0)
+    (property "Footprint" "Diode_THT:D_DO-35_SOD27_P3.81mm_Vertical_AnodeUp" (id 2) (at 198.755 95.25 0)
       (effects (font (size 1.27 1.27)) hide)
     )
@@
       (effects (font (size 1.27 1.27)) (justify right) hide)
     )
-    (property "Footprint" "Diode_THT:D_DO-35_SOD27_P7.62mm_Horizontal" (id 2) (at 206.375 52.07 0)
+    (property "Footprint" "Diode_THT:D_DO-35_SOD27_P3.81mm_Vertical_AnodeUp" (id 2) (at 206.375 52.07 0)
       (effects (font (size 1.27 1.27)) hide)
     )
@@
       (effects (font (size 1.27 1.27)) (justify right) hide)
     )
-    (property "Footprint" "Diode_THT:D_DO-35_SOD27_P7.62mm_Horizontal" (id 2) (at 179.705 95.25 0)
+    (property "Footprint" "Diode_THT:D_DO-35_SOD27_P3.81mm_Vertical_AnodeUp" (id 2) (at 179.705 95.25 0)
       (effects (font (size 1.27 1.27)) hide)
     )
@@
       (effects (font (size 1.27 1.27)) (justify right) hide)
     )
-    (property "Footprint" "Diode_THT:D_DO-35_SOD27_P7.62mm_Horizontal" (id 2) (at 206.375 73.66 0)
+    (property "Footprint" "Diode_THT:D_DO-35_SOD27_P3.81mm_Vertical_AnodeUp" (id 2) (at 206.375 73.66 0)
       (effects (font (size 1.27 1.27)) hide)
     )
@@
     )
     (path "/3c157981-87c5-4c53-8982-7356b0394275"
-      (reference "D1") (unit 1) (value "1N914") (footprint "Diode_THT:D_DO-35_SOD27_P7.62mm_Horizontal")
+      (reference "D1") (unit 1) (value "1N914") (footprint "Diode_THT:D_DO-35_SOD27_P3.81mm_Vertical_AnodeUp")
     )
     (path "/e5c48d92-898f-4d96-a8a1-acda90e87277"
@@
     )
     (path "/855cd4c5-6326-48ed-b5a5-0a56b3dbfb10"
-      (reference "D3") (unit 1) (value "1N914") (footprint "Diode_THT:D_DO-35_SOD27_P7.62mm_Horizontal")
+      (reference "D3") (unit 1) (value "1N914") (footprint "Diode_THT:D_DO-35_SOD27_P3.81mm_Vertical_AnodeUp")
     )
     (path "/bb17bd9f-4510-4a70-8c2f-5e656b5a613f"
-      (reference "D4") (unit 1) (value "1N914") (footprint "Diode_THT:D_DO-35_SOD27_P7.62mm_Horizontal")
+      (reference "D4") (unit 1) (value "1N914") (footprint "Diode_THT:D_DO-35_SOD27_P3.81mm_Vertical_AnodeUp")
     )
     (path "/3cab11c8-cea2-4f66-b64a-ee8170e16031"
-      (reference "D5") (unit 1) (value "1N914") (footprint "Diode_THT:D_DO-35_SOD27_P7.62mm_Horizontal")
+      (reference "D5") (unit 1) (value "1N914") (footprint "Diode_THT:D_DO-35_SOD27_P3.81mm_Vertical_AnodeUp")
     )
     (path "/08307301-b756-4307-9a1b-022a72b58ba8"
-      (reference "D6") (unit 1) (value "1N914") (footprint "Diode_THT:D_DO-35_SOD27_P7.62mm_Horizontal")
+      (reference "D6") (unit 1) (value "1N914") (footprint "Diode_THT:D_DO-35_SOD27_P3.81mm_Vertical_AnodeUp")
     )
     (path "/6f05b559-0df4-4d0b-b671-a4863708506c"
-      (reference "D7") (unit 1) (value "1N914") (footprint "Diode_THT:D_DO-35_SOD27_P7.62mm_Horizontal")
+      (reference "D7") (unit 1) (value "1N914") (footprint "Diode_THT:D_DO-35_SOD27_P3.81mm_Vertical_AnodeUp")
     )
     (path "/e1bde1ce-78a8-46ed-a1cd-0ae2a256c2de"
-      (reference "D8") (unit 1) (value "1N914") (footprint "Diode_THT:D_DO-35_SOD27_P7.62mm_Horizontal")
+      (reference "D8") (unit 1) (value "1N914") (footprint "Diode_THT:D_DO-35_SOD27_P3.81mm_Vertical_AnodeUp")
     )
     (path "/bdf5c1ae-9059-4e28-9217-b6cc23c4449a"
-      (reference "D9") (unit 1) (value "1N914") (footprint "Diode_THT:D_DO-35_SOD27_P7.62mm_Horizontal")
+      (reference "D9") (unit 1) (value "1N914") (footprint "Diode_THT:D_DO-35_SOD27_P3.81mm_Vertical_AnodeUp")
     )
     (path "/2c92f753-a2c2-4985-b4b4-1278afff8575"
-      (reference "D10") (unit 1) (value "1N914") (footprint "Diode_THT:D_DO-35_SOD27_P7.62mm_Horizontal")
+      (reference "D10") (unit 1) (value "1N914") (footprint "Diode_THT:D_DO-35_SOD27_P3.81mm_Vertical_AnodeUp")
     )
     (path "/8e5dd52a-e27a-41fb-b0ab-24b3ea21250f"
-      (reference "D11") (unit 1) (value "1N914") (footprint "Diode_THT:D_DO-35_SOD27_P7.62mm_Horizontal")
+      (reference "D11") (unit 1) (value "1N914") (footprint "Diode_THT:D_DO-35_SOD27_P3.81mm_Vertical_AnodeUp")
     )
     (path "/3be4026d-8822-4555-89da-7ddf08ab9e9b"
-      (reference "D12") (unit 1) (value "1N914") (footprint "Diode_THT:D_DO-35_SOD27_P7.62mm_Horizontal")
+      (reference "D12") (unit 1) (value "1N914") (footprint "Diode_THT:D_DO-35_SOD27_P3.81mm_Vertical_AnodeUp")
     )
     (path "/34518b74-2692-4857-b7a6-a3054b6fd2eb"
